File: gerador_sinais.sch (KiCad schematic (older format))
At the start: 18 parts

Commit message: Add valores aos componentes
Parts:
- removed R?: R, symbol R
- added R?: 68K, symbol R
- C? (x2): value C -> 10 n
- R?: value R -> RK
- R?: value R -> 5K
- R? (x2): value R -> 33K
- R?: value R -> K
Connections:
- net labels added: V1, V2
- wire segments 46 -> 47
Other:
- note added: "Amplificador não Inversor\n"
- note added: "Circuito Integrador\n"
- note added: "Ponte de Wien ( Gera onda Senoidal)\n"
- note added: "Trigger Schimit\n"
Changed lines of the file:
@@
 LIBS:contrib
 LIBS:valves
+LIBS:gerador_sinais-cache
 EELAYER 25 0
 EELAYER END
@@
 P 2050 3800
 F 0 "R?" V 2130 3800 50  0000 C CNN
-F 1 "R" V 2050 3800 50  0000 C CNN
+F 1 "RK" V 2050 3800 50  0000 C CNN
 F 2 "" V 1980 3800 50  0001 C CNN
 F 3 "" H 2050 3800 50  0001 C CNN
@@
 P 2400 3550
 F 0 "R?" V 2480 3550 50  0000 C CNN
-F 1 "R" V 2400 3550 50  0000 C CNN
+F 1 "5K" V 2400 3550 50  0000 C CNN
 F 2 "" V 2330 3550 50  0001 C CNN
 F 3 "" H 2400 3550 50  0001 C CNN
@@
 P 1750 3250
 F 0 "C?" H 1775 3350 50  0000 L CNN
-F 1 "C" H 1775 3150 50  0000 L CNN
+F 1 "10 n" H 1775 3150 50  0000 L CNN
 F 2 "" H 1788 3100 50  0001 C CNN
 F 3 "" H 1750 3250 50  0001 C CNN
@@
 P 1400 3200
 F 0 "R?" V 1480 3200 50  0000 C CNN
-F 1 "R" V 1400 3200 50  0000 C CNN
+F 1 "33K" V 1400 3200 50  0000 C CNN
 F 2 "" V 1330 3200 50  0001 C CNN
 F 3 "" H 1400 3200 50  0001 C CNN
@@
 P 1450 2550
 F 0 "C?" H 1475 2650 50  0000 L CNN
-F 1 "C" H 1475 2450 50  0000 L CNN
+F 1 "10 n" H 1475 2450 50  0000 L CNN
 F 2 "" H 1488 2400 50  0001 C CNN
 F 3 "" H 1450 2550 50  0001 C CNN
@@
 P 1900 2300
 F 0 "R?" V 1980 2300 50  0000 C CNN
-F 1 "R" V 1900 2300 50  0000 C CNN
+F 1 "33K" V 1900 2300 50  0000 C CNN
 F 2 "" V 1830 2300 50  0001 C CNN
 F 3 "" H 1900 2300 50  0001 C CNN
@@
 $Comp
 L R R?
-U 1 1 5935DACE
-P 3400 2850
-F 0 "R?" V 3480 2850 50  0000 C CNN
-F 1 "R" V 3400 2850 50  0000 C CNN
-F 2 "" V 3330 2850 50  0001 C CNN
-F 3 "" H 3400 2850 50  0001 C CNN
-	1    3400 2850
-	0    1    1    0
-$EndComp
-Wire Wire Line
-	3550 2850 4300 2850
-Wire Wire Line
-	3850 2850 3850 2400
-Wire Wire Line
-	3850 2400 4500 2400
-Connection ~ 3850 2850
-$Comp
-L R R?
 U 1 1 5935DB88
 P 4650 2400
 F 0 "R?" V 4730 2400 50  0000 C CNN
-F 1 "R" V 4650 2400 50  0000 C CNN
+F 1 "K" V 4650 2400 50  0000 C CNN
 F 2 "" V 4580 2400 50  0001 C CNN
 F 3 "" H 4650 2400 50  0001 C CNN
@@
 	9050 2500 9050 3000
 Wire Wire Line
-	8850 3000 9250 3000
+	8850 3000 9550 3000
 Connection ~ 9050 3000
 $Comp
@@
 Wire Notes Line
 	9400 4400 7700 4400
+Text Notes 1650 4350 0    60   ~ 12
+Ponte de Wien ( Gera onda Senoidal)\n
+Text Notes 4600 4300 0    60   ~ 12
+Trigger Schimit\n
+Text Notes 6200 4300 0    60   ~ 12
+Circuito Integrador\n
+Text Notes 8000 4300 0    60   ~ 12
+Amplificador não Inversor\n
+Text HLabel 5150 2850 1    60   Input ~ 0
+V2
+Text HLabel 3500 2850 1    60   Input ~ 0
+V1
+Wire Wire Line
+	4500 2400 4150 2400
+Wire Wire Line
+	4150 2400 4150 2850
+Connection ~ 4150 2850
+Wire Wire Line
+	3250 2850 3800 2850
+$Comp
+L R R?
+U 1 1 593627EF
+P 3950 2850
+F 0 "R?" V 4030 2850 50  0000 C CNN
+F 1 "68K" V 3950 2850 50  0000 C CNN
+F 2 "" V 3880 2850 50  0001 C CNN
+F 3 "" H 3950 2850 50  0001 C CNN
+	1    3950 2850
+	0    1    1    0
+$EndComp
+Wire Wire Line
+	4100 2850 4300 2850
 $EndSCHEMATC
